File: ESP_Cam_recap.kicad_sch (KiCad schematic)
At the start: 8 parts, among them U1 ESP32-S3FN8

Commit message: power section und clock
Parts:
- added C13: 1nF, symbol Device:C_Small
- added C14: 0.1uF, symbol Device:C_Small
- added C9: 1uF, symbol Device:C_Small
- added R12, R4: 10k, symbol Device:R_Small
- added R13: 0, symbol Device:R_Small
- added Y1: ECS-2532HS-400-3-G-TR, ECS2532HS4003GTR, symbol SamacSys_Parts:ECS-2532HS-400-3-G-TR
Connections:
- net GND: now also C14.2, C9.2, Y1.2 (GROUND)
- net VDD3P3: now also R12.1
- net at U1.4 (CHIP_PU/RESET): now also C9.1, R4.1
- net at U1.54 (XTAL_P): now also C13.2
- new net: R13.2, Y1.3 (OUTPUT)
- new net: C14.1, R12.2, Y1.4 (VDD)
- new net: C13.1, R13.1
- new net PG: R4.2
- no-connect marks 2 -> 7
Other:
- note added: "0402 or 0603 (Swap with 22ohm if needed)"
- note added: "Power good w delay"
- note added: "info zu xtal_N/P in field 11(doppelklick auf esc)"

Commit message: finished schematics
Parts:
- added J1: USB_B_Micro, symbol Connector:USB_B_Micro
- added J2: Micro_SD_Card, symbol Connector:Micro_SD_Card
- added R14, R15, R16, R17, R18, R19, R20, R21, R22, R23: 10k, symbol Device:R_Small
- added SW2: SW_Push, symbol Switch:SW_Push
Connections:
- net GND: now also J1.5 (GND), J1.6 (Shield), J2.6 (VSS), J2.9 (SHIELD), R14.2, R21.2, R23.2
- net USB_N: now reaches U1.25 (GPIO19/USB_D-/ADC2_CH8)
- net USB_N: now also J1.2 (D-)
- net USB_P: now reaches U1.26 (GPIO20/USB_D+/ADC2_CH9)
- net USB_P: now also J1.3 (D+)
- net SD_D2: now reaches U1.38 (GPIO33)
- net SD_D2: now also J2.1 (DAT2), R15.2
- net SD_D3: now reaches U1.39 (GPIO34)
- net SD_D3: now also J2.2 (DAT3/CD), R16.2
- net SD_CMD: now reaches U1.40 (GPIO35)
- net SD_CMD: now also J2.3 (CMD), R17.2
- net SD_CLK: now reaches U1.41 (GPIO36)
- net SD_CLK: now also J2.5 (CLK), R18.2
- net SD_D0: now reaches U1.42 (GPIO37)
- net SD_D0: now also J2.7 (DAT0), R19.2
- net SD_D1: now reaches U1.43 (GPIO38)
- net SD_D1: now also J2.8 (DAT1), R20.2
- net at U1.5 (GPIO0/BOOT): now also R22.2, SW2.1
- net at U1.51 (GPIO45): now also R23.1
- net at U1.52 (GPIO46): now also R21.1
- net VDD3P3 renamed +3V3
- net +3V3: now also J2.4 (VDD), R15.1, R16.1, R17.1, R18.1, R19.1, R20.1, R22.1
- new net: R14.1, SW2.2
- new net VUSB: J1.1 (VBUS)
- no-connect marks 7 -> 40
Other:
- note added: "Keine Ahnung ob das funktioniert!"
- note added: "silk prog"

Commit message: cam
Parts:
- removed D1: DESD3V3E1BL, Diode_SMD:D_SOD-882, symbol Diode:ESD9B3.3ST5G
- added D1: SP0402B-ELC-01ETG, SamacSys_Parts2:SP0402BELC01ETG, symbol SamacSys_Parts2:SP0402B-ELC-01ETG
- C1, C13, C14, C2, C3, C4, C5, C6, C9: footprint (none) -> Capacitor_SMD:C_0201_0603Metric
- J1: footprint (none) -> Connector_USB:USB_Micro-AB_Molex_47590-0001
- J2: footprint (none) -> Connector_Card:microSD_HC_Molex_47219-2001
- R12, R13, R14, R15, R16, R17, R18, R19, R20, R21, R22, R23, R4: footprint (none) -> Resistor_SMD:R_0201_0603Metric
- SW2: footprint (none) -> Button_Switch_SMD:SW_SPST_EVQP2_ShortPushTravel_H2.5mm
- Y1: footprint ECS2532HS4003GTR -> SamacSys_Parts2:ECS2532HS4003GTR
Connections:
- net +3V3: no longer C1.1
- net GND: now also D1.1
- net XTAL_P: now reaches C13.2, U1.54 (XTAL_P)
- net I2C_SCL: now reaches U1.10 (GPIO5/ADC1_CH4)
- net DVP_VSYNC: now reaches U1.11 (GPIO6/ADC1_CH5)
- net DVP_HREF: now reaches U1.12 (GPIO7/ADC1_CH6)
- net DVP_Y4: now reaches U1.13 (GPIO8/ADC1_CH7)
- net DVP_Y3: now reaches U1.14 (GPIO9/ADC1_CH8)
- net DVP_Y5: now reaches U1.15 (GPIO10/ADC1_CH9)
- net DVP_Y2: now reaches U1.16 (GPIO11/ADC2_CH0)
- net DVP_Y6: now reaches U1.17 (GPIO12/ADC2_CH1)
- net DVP_PCLK: now reaches U1.18 (GPIO13/ADC2_CH2)
- net XMCLK: now reaches U1.21 (GPIO15/ADC2_CH4/XTAL_32K_P)
- net DVP_Y9: now reaches U1.22 (GPIO16/ADC2_CH5/XTAL_32K_N)
- net DVP_Y8: now reaches U1.23 (GPIO17/ADC2_CH6)
- net DVP_Y7: now reaches U1.24 (GPIO18/ADC2_CH7)
- net I2C_SDA: now reaches U1.9 (GPIO4/ADC1_CH3)
- net VUSB renamed +5V
- net +5V: now also C1.1, D1.2
- no-connect marks 40 -> 26
Other:
- added sheet Cam (cam.kicad_sch)
- note added: "close to usb port"
- note added: "info zu xtal_N/P in field 11(doppelklick auf esc32)"
- note removed: "Keine Ahnung ob das funktioniert!"
- note removed: "info zu xtal_N/P in field 11(doppelklick auf esc)"
- moved on the sheet: C1, C13, C14, C2, C3, C4, C5, C6, C9, J1, J2, R12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
