File: power.kicad_sch (KiCad schematic)
At the start: 22 parts, among them IC1 TPS629206QDRLRQ1, IC2 BQ24074RGTR, SW1 SW_Nidec_CAS-120A1

Commit message: cam
Parts:
- added C15, C16, C17, C18: 1uF, Capacitor_SMD:C_0201_0603Metric, symbol Device:C_Small
- added IC3: LP5912Q1.5DRVRQ1, SamacSys_Parts2:SON65P200X200X80-7N, symbol DONTMIGRATE:LP5912Q1.5DRVRQ1
- added IC4: LP5912Q2.8DRVRQ1, SamacSys_Parts2:SON65P200X200X80-7N, symbol DONTMIGRATE:LP5912Q2.8DRVRQ1
- added R2: BATT_CON, Resistor_SMD:R_2512_6332Metric_Pad1.40x3.35mm_HandSolder, symbol Device:R_Small
- added R6: 18k, Resistor_SMD:R_0201_0603Metric, symbol Device:R_Small
- C10: footprint (none) -> Capacitor_SMD:C_0201_0603Metric
- C7: renamed from C12; footprint (none) -> Capacitor_SMD:C_0201_0603Metric
- C8: renamed from C11; footprint (none) -> Capacitor_SMD:C_0201_0603Metric
- D2: renamed from D5; footprint (none) -> LED_SMD:LED_0402_1005Metric
- D3: renamed from D4; footprint (none) -> LED_SMD:LED_0402_1005Metric
- D4: renamed from D2; footprint (none) -> LED_SMD:LED_0402_1005Metric
- IC1: renamed from IC2; footprint QFN50P300X300X100-17N-D -> SamacSys_Parts2:QFN50P300X300X100-17N-D; Field11 https://www.ti.com/lit/ds/symlink/bq24074.pdf?ts=1763244263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 -> (none)
- IC2: renamed from IC1; footprint SOTFL50P160X60-8N -> SamacSys_Parts2:SOTFL50P160X60-8N
- R1: renamed from R9; footprint (none) -> Resistor_SMD:R_0201_0603Metric
- R10: renamed from R1; footprint (none) -> Resistor_SMD:R_0201_0603Metric
- R11: renamed from R2; footprint (none) -> Resistor_SMD:R_0201_0603Metric
- R24: renamed from R5; footprint (none) -> Resistor_SMD:R_0201_0603Metric
- R25: renamed from R3; footprint (none) -> Resistor_SMD:R_0201_0603Metric
- R3: renamed from R10; value 4.12k -> 3.05k; footprint (none) -> Resistor_SMD:R_0201_0603Metric; now not fitted
- R5: renamed from R11; value 1.13k -> 1.78k; footprint (none) -> Resistor_SMD:R_0201_0603Metric
- R7: footprint (none) -> Resistor_SMD:R_0201_0603Metric
- R8: value 1.18k -> 3.44k; footprint (none) -> Resistor_SMD:R_0201_0603Metric
- R9: renamed from R6; footprint (none) -> Resistor_SMD:R_0201_0603Metric
- renumbered C8 to C11, C7 to C12
Connections:
- net BQOUT: now also IC2.7 (EN); no longer SW1.1 (C)
- net CHG: now reaches D2.1 (K), IC1.9 (~{CHG})
- net +BATT: now reaches SW1.2 (B)
- net +BATT: now also C7.1, R2.1; no longer IC2.7 (EN)
- net at SW1.3 (A): now also IC1.2 (BAT_1), IC1.3 (BAT_2)
- net at IC2.4 (SW), L1.2: no longer IC2.3 (VOS)
- net GND renamed -BATT
- net -BATT: now also C15.2, C16.2, C17.2, C18.2, IC3.5 (GND), IC3.7 (EP), IC4.5 (GND_1), IC4.7 (GND_2), R2.2, R6.1; no longer IC1.14 (TMR)
- removed net VBAT: C7.1, IC1.2 (BAT_1), IC1.3 (BAT_2)
- net VOUT33 renamed +3V3
- net +3V3: now also IC2.3 (VOS), C15.1, C17.1, IC3.4 (EN), IC3.6 (IN), IC4.4 (EN), IC4.6 (IN)
- net VUSB renamed +5V
- new net: IC1.14 (TMR), R6.2
- new net +1V5: C16.1, IC3.1 (OUT)
- new net +2V8: C18.1, IC4.1 (OUT)
- no-connect marks 1 -> 3
Other:
- note added: "1.5V Voltage supply"
- note added: "2.8V Voltage supply"
- note added: "Battery management"
- note removed: "RECALC Page 34"
- moved on the sheet: C10, C11, C12, C7, C8, D2, D3, D4, IC1, IC2, L1, R1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
